File: electrium-esc/electrium-esc.kicad_sch (KiCad schematic)
At the start: 7 parts

Commit message: Prototype (almost) finished
Have to do electric check rules
Parts:
- added C?: 100n, symbol Device:C
- added D? (x2): LED, symbol Device:LED
- added J?: Conn_01x04_Male, symbol Connector:Conn_01x04_Male
- added J?: Conn_01x03_Male, symbol Connector:Conn_01x03_Male
- added R? (x4): SHUNT, symbol Device:R
- added R? (x2): 0, symbol Device:R
- added R? (x2): 2k2, symbol Device:R
- added R?: 100, symbol Device:R
Connections:
- net +5V: now also J?.2 (Pin_2)
- net GND: now also C?.2, D?.1 (K), D?.1 (K), J?.3 (Pin_3), J?.4 (Pin_4), R?.2, R?.2, R?.2, R?.2
- net MCU (STM32F407ZGT6)/GPIO1: now also R?.2
- net MCU (STM32F407ZGT6)/GPIO2: now also R?.2
- net MCU (STM32F407ZGT6)/SERVO: now also C?.1, R?.1
- new net: D?.2 (A), R?.1 (x2)
- new net: J?.3 (Pin_3), R?.1
- new net: J?.2 (Pin_2), R?.1
- new net: J?.1 (Pin_1), R?.2
- new net +3.3V: J?.1 (Pin_1), R?.2
- new net MCU (STM32F407ZGT6)/LED: R?.2
- new net Motor Driver A (DRV8301)/H1_LOW: R?.1
- new net Motor Driver A (DRV8301)/H3_LOW: R?.1
- new net Motor Driver B (DRV8301)/H1_LOW: R?.1
- new net Motor Driver B (DRV8301)/H3_LOW: R?.1
Other:
- added sheet Power MOSFETs1 (MOSFETs.kicad_sch)
- sheet MCU (STM32F407ZGT6) ports: added CS_A, CS_B, LED; removed none
- sheet Motor Driver A (DRV8301) ports: added H1_LOW, H1_VS, H2_LOW, H2_VS, H3_LOW, H3_VS, M_H1, M_H2, M_H3, M_L1, M_L2, M_L3, SCS, SH1_A, SH1_B, SH2_A, SH2_B; removed none
- sheet Motor Driver B (DRV8301) ports: added H1_LOW, H1_VS, H2_LOW, H2_VS, H3_LOW, H3_VS, M_H1, M_H2, M_H3, M_L1, M_L2, M_L3, SCS, SH1_A, SH1_B, SH2_A, SH2_B; removed none
- sheet Power MOSFETs ports: added H1_LOW, H1_VS, H2_LOW, H2_VS, H3_LOW, H3_VS, M_H1, M_H2, M_H3, M_L1, M_L2, M_L3, Phase_1, Phase_2, Phase_3; removed none
