File: electrium-esc/electrium-esc.kicad_sch (KiCad schematic)
At the start: 32 parts, among them J2 USB_MICRO, J3 Conn_01x04_Male, J4 Conn_01x03_Male, J5 Conn_01x04_Male

Commit message: Update diodes (real version now)
Parts:
- removed D3, D4: D_Shockley, Diode_SMD:D_0603_1608Metric, symbol Device:D_Shockley
- added D3, D4: 1N5819, Diode_THT:D_DO-41_SOD81_P10.16mm_Horizontal, symbol Diode:1N5819
- J4: value Conn_01x03_Male -> SERVO
Connections:
- net +3.3V: now also D4.1 (K)
- net AN_IN: now also D3.1 (K), D4.2 (A)
- net GND: now also D3.2 (A)
Changed lines of the file:
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@@
   (junction (at 238.76 25.4) (diameter 0) (color 0 0 0 0)
   )
-  (junction (at 40.64 38.1) (diameter 0) (color 0 0 0 0)
-  )
   (junction (at 214.63 90.17) (diameter 0) (color 0 0 0 0)
   )
@@
   (junction (at 78.74 161.29) (diameter 0) (color 0 0 0 0)
   )
+  (junction (at 36.83 38.1) (diameter 0) (color 0 0 0 0)
+  )
   (junction (at 254 25.4) (diameter 0) (color 0 0 0 0)
   )
   (junction (at 81.28 55.88) (diameter 0) (color 0 0 0 0)
   )
+  (junction (at 58.42 29.21) (diameter 0) (color 0 0 0 0)
+  )
+  (junction (at 58.42 38.1) (diameter 0) (color 0 0 0 0)
+  )
   (junction (at 207.01 72.39) (diameter 0) (color 0 0 0 0)
   )
@@
   )
   (junction (at 207.01 74.93) (diameter 0) (color 0 0 0 0)
-  )
-  (junction (at 60.96 38.1) (diameter 0) (color 0 0 0 0)
   )
   (junction (at 214.63 154.94) (diameter 0) (color 0 0 0 0)
@@
     (stroke (width 0) (type default) (color 0 0 0 0))
   )
+  (wire (pts (xy 36.83 29.21) (xy 36.83 38.1))
+    (stroke (width 0) (type default) (color 0 0 0 0))
+  )
   (wire (pts (xy 198.12 67.31) (xy 214.63 67.31))
     (stroke (width 0) (type default) (color 0 0 0 0))
@@
     (stroke (width 0) (type default) (color 0 0 0 0))
   )
+  (wire (pts (xy 41.91 29.21) (xy 36.83 29.21))
+    (stroke (width 0) (type default) (color 0 0 0 0))
+  )
   (wire (pts (xy 198.12 142.24) (xy 201.93 142.24))
     (stroke (width 0) (type default) (color 0 0 0 0))
   )
+  (wire (pts (xy 36.83 38.1) (xy 45.72 38.1))
+    (stroke (width 0) (type default) (color 0 0 0 0))
+  )
   (wire (pts (xy 165.1 162.56) (xy 168.91 162.56))
     (stroke (width 0) (type default) (color 0 0 0 0))
   )
-  (wire (pts (xy 60.96 29.21) (xy 60.96 38.1))
+  (wire (pts (xy 58.42 29.21) (xy 58.42 38.1))
     (stroke (width 0) (type default) (color 0 0 0 0))
   )
@@
     (stroke (width 0) (type default) (color 0 0 0 0))
   )
-  (wire (pts (xy 40.64 38.1) (xy 34.29 38.1))
+  (wire (pts (xy 34.29 38.1) (xy 36.83 38.1))
     (stroke (width 0) (type default) (color 0 0 0 0))
   )
@@
     (stroke (width 0) (type default) (color 0 0 0 0))
   )
-  (wire (pts (xy 66.04 38.1) (xy 60.96 38.1))
+  (wire (pts (xy 53.34 38.1) (xy 58.42 38.1))
     (stroke (width 0) (type default) (color 0 0 0 0))
   )
@@
     (stroke (width 0) (type default) (color 0 0 0 0))
   )
+  (wire (pts (xy 49.53 29.21) (xy 58.42 29.21))
+    (stroke (width 0) (type default) (color 0 0 0 0))
+  )
   (wire (pts (xy 220.98 92.71) (xy 214.63 92.71))
     (stroke (width 0) (type default) (color 0 0 0 0))
@@
     (stroke (width 0) (type default) (color 0 0 0 0))
   )
-  (wire (pts (xy 48.26 29.21) (xy 53.34 29.21))
-    (stroke (width 0) (type default) (color 0 0 0 0))
-  )
   (wire (pts (xy 198.12 104.14) (xy 226.06 104.14))
     (stroke (width 0) (type default) (color 0 0 0 0))
@@
     (stroke (width 0) (type default) (color 0 0 0 0))
   )
-  (wire (pts (xy 40.64 29.21) (xy 40.64 38.1))
-    (stroke (width 0) (type default) (color 0 0 0 0))
-  )
   (wire (pts (xy 198.12 44.45) (xy 224.79 44.45))
     (stroke (width 0) (type default) (color 0 0 0 0))
@@
     (stroke (width 0) (type default) (color 0 0 0 0))
   )
+  (wire (pts (xy 58.42 29.21) (xy 64.77 29.21))
+    (stroke (width 0) (type default) (color 0 0 0 0))
+  )
   (wire (pts (xy 152.4 125.73) (xy 167.64 125.73))
     (stroke (width 0) (type default) (color 0 0 0 0))
@@
     (stroke (width 0) (type default) (color 0 0 0 0))
   )
-  (wire (pts (xy 60.96 38.1) (xy 53.34 38.1))
-    (stroke (width 0) (type default) (color 0 0 0 0))
-  )
   (wire (pts (xy 152.4 102.87) (xy 167.64 102.87))
     (stroke (width 0) (type default) (color 0 0 0 0))
@@
     (stroke (width 0) (type default) (color 0 0 0 0))
   )
+  (wire (pts (xy 72.39 29.21) (xy 76.2 29.21))
+    (stroke (width 0) (type default) (color 0 0 0 0))
+  )
   (wire (pts (xy 198.12 132.08) (xy 220.98 132.08))
     (stroke (width 0) (type default) (color 0 0 0 0))
@@
     (stroke (width 0) (type default) (color 0 0 0 0))
   )
+  (wire (pts (xy 58.42 38.1) (xy 66.04 38.1))
+    (stroke (width 0) (type default) (color 0 0 0 0))
+  )
   (wire (pts (xy 152.4 165.1) (xy 157.48 165.1))
     (stroke (width 0) (type default) (color 0 0 0 0))
@@
   )
   (wire (pts (xy 209.55 147.32) (xy 209.55 144.78))
-    (stroke (width 0) (type default) (color 0 0 0 0))
-  )
-  (wire (pts (xy 45.72 38.1) (xy 40.64 38.1))
     (stroke (width 0) (type default) (color 0 0 0 0))
   )
@@
     (pin "1")
   )
-  (symbol (lib_id "Device:D_Shockley") (at 57.15 29.21 180) (unit 1)
-    (in_bom yes) (on_board yes)
-    (property "Reference" "D4" (id 0) (at 57.15 26.67 0))
-    (property "Value" "D_Shockley" (id 1) (at 67.31 29.21 0))
-    (property "Footprint" "Diode_SMD:D_0603_1608Metric" (id 2) (at 57.15 29.21 0)
-      (effects (font (size 1.27 1.27)) hide)
-    )
-    (property "Datasheet" "~" (id 3) (at 57.15 29.21 0)
-      (effects (font (size 1.27 1.27)) hide)
-    )
-    (pin "1")
-    (pin "2")
-  )
   (symbol (lib_id "Device:R") (at 207.01 78.74 0) (unit 1)
     (in_bom yes) (on_board yes)
@@
     )
     (pin "1")
+  )
+  (symbol (lib_id "Diode:1N5819") (at 45.72 29.21 180) (unit 1)
+    (in_bom yes) (on_board yes)
+    (property "Reference" "D3" (id 0) (at 41.91 26.67 0))
+    (property "Value" "1N5819" (id 1) (at 41.91 31.75 0))
+    (property "Footprint" "Diode_THT:D_DO-41_SOD81_P10.16mm_Horizontal" (id 2) (at 45.72 24.765 0)
+      (effects (font (size 1.27 1.27)) hide)
+    )
+    (property "Datasheet" "http://www.vishay.com/docs/88525/1n5817.pdf" (id 3) (at 45.72 29.21 0)
+      (effects (font (size 1.27 1.27)) hide)
+    )
+    (pin "1")
+    (pin "2")
   )
   (symbol (lib_id "power:GND") (at 71.12 168.91 0) (unit 1)
@@
     (pin "4")
   )
+  (symbol (lib_id "Diode:1N5819") (at 68.58 29.21 180) (unit 1)
+    (in_bom yes) (on_board yes)
+    (property "Reference" "D4" (id 0) (at 64.77 26.67 0))
+    (property "Value" "1N5819" (id 1) (at 64.77 31.75 0))
+    (property "Footprint" "Diode_THT:D_DO-41_SOD81_P10.16mm_Horizontal" (id 2) (at 68.58 24.765 0)
+      (effects (font (size 1.27 1.27)) hide)
+    )
+    (property "Datasheet" "http://www.vishay.com/docs/88525/1n5817.pdf" (id 3) (at 68.58 29.21 0)
+      (effects (font (size 1.27 1.27)) hide)
+    )
+    (pin "1")
+    (pin "2")
+  )
   (symbol (lib_id "power:+5V") (at 66.04 157.48 0) (unit 1)
     (in_bom yes) (on_board yes) (fields_autoplaced)
@@
     (pin "1")
   )
+  (symbol (lib_id "power:+3.3V") (at 76.2 29.21 270) (unit 1)
+    (in_bom yes) (on_board yes)
+    (property "Reference" "#PWR078" (id 0) (at 72.39 29.21 0)
+      (effects (font (size 1.27 1.27)) hide)
+    )
+    (property "Value" "+3.3V" (id 1) (at 76.2 31.75 90))
+    (property "Footprint" "" (id 2) (at 76.2 29.21 0)
+      (effects (font (size 1.27 1.27)) hide)
+    )
+    (property "Datasheet" "" (id 3) (at 76.2 29.21 0)
+      (effects (font (size 1.27 1.27)) hide)
+    )
+    (pin "1")
+  )
   (symbol (lib_id "Device:LED") (at 118.11 182.88 90) (unit 1)
     (in_bom yes) (on_board yes) (fields_autoplaced)
@@
     )
     (pin "1")
-  )
-  (symbol (lib_id "Device:D_Shockley") (at 44.45 29.21 0) (unit 1)
-    (in_bom yes) (on_board yes)
-    (property "Reference" "D3" (id 0) (at 44.45 26.67 0))
-    (property "Value" "D_Shockley" (id 1) (at 34.29 29.21 0))
-    (property "Footprint" "Diode_SMD:D_0603_1608Metric" (id 2) (at 44.45 29.21 0)
-      (effects (font (size 1.27 1.27)) hide)
-    )
-    (property "Datasheet" "~" (id 3) (at 44.45 29.21 0)
-      (effects (font (size 1.27 1.27)) hide)
-    )
-    (pin "1")
-    (pin "2")
   )
   (symbol (lib_id "Device:R") (at 161.29 162.56 270) (unit 1)
@@
     (in_bom yes) (on_board yes)
     (property "Reference" "J4" (id 0) (at 53.34 156.21 0))
-    (property "Value" "Conn_01x03_Male" (id 1) (at 53.34 158.75 0))
+    (property "Value" "SERVO" (id 1) (at 53.34 158.75 0))
     (property "Footprint" "Connector_PinHeader_2.54mm:PinHeader_1x03_P2.54mm_Vertical" (id 2) (at 58.42 163.83 0)
       (effects (font (size 1.27 1.27)) hide)
@@
       (reference "#PWR077") (unit 1) (value "GND") (footprint "")
     )
+    (path "/7edd22c2-7370-48d7-af32-c9d630dfd47e"
+      (reference "#PWR078") (unit 1) (value "+3.3V") (footprint "")
+    )
     (path "/95515899-f309-4706-b478-ef0c1d74de3d/6e926fcb-bc57-4a6a-ac9a-7920661fd921"
       (reference "C1") (unit 1) (value "4.7u") (footprint "Capacitor_SMD:C_0603_1608Metric")
@@
       (reference "D2") (unit 1) (value "1N5819") (footprint "Diode_THT:D_DO-41_SOD81_P10.16mm_Horizontal")
     )
-    (path "/8fd51e59-8aaf-459c-8449-142ad8ed12b0"
-      (reference "D3") (unit 1) (value "D_Shockley") (footprint "Diode_SMD:D_0603_1608Metric")
-    )
-    (path "/02300329-aad1-4f53-b5c5-b1e6b0276df0"
-      (reference "D4") (unit 1) (value "D_Shockley") (footprint "Diode_SMD:D_0603_1608Metric")
+    (path "/3c103bef-0efb-4142-b313-3083a43ce99d"
+      (reference "D3") (unit 1) (value "1N5819") (footprint "Diode_THT:D_DO-41_SOD81_P10.16mm_Horizontal")
+    )
+    (path "/7c2a1523-547e-41f9-846d-b97ecea82980"
+      (reference "D4") (unit 1) (value "1N5819") (footprint "Diode_THT:D_DO-41_SOD81_P10.16mm_Horizontal")
     )
     (path "/5098eb75-ab3f-49e8-b692-4372bb393d18"
@@
     )
     (path "/9797036c-f702-4f5f-bef1-41a9950c6932"
-      (reference "J4") (unit 1) (value "Conn_01x03_Male") (footprint "Connector_PinHeader_2.54mm:PinHeader_1x03_P2.54mm_Vertical")
+      (reference "J4") (unit 1) (value "SERVO") (footprint "Connector_PinHeader_2.54mm:PinHeader_1x03_P2.54mm_Vertical")
     )
     (path "/928f53cb-3848-4c94-9638-22c4359c3f9a"

Commit message: Update more components and few traces
Final design hopefully done by tomorrow. Logistical problems are coming through, needs to suit components to those needs
Parts:
- removed J3: Conn_01x04_Male, Connector_PinHeader_2.54mm:PinHeader_1x04_P2.54mm_Vertical, symbol Connector:Conn_01x04_Male
- D3, D4: footprint Diode_THT:D_DO-41_SOD81_P10.16mm_Horizontal -> Diode_SMD:D_0603_1608Metric
Connections:
- no-connect marks 2 -> 4
Other:
- removed sheet CAN Bus

Commit message: Add power connections
I realize Vias are unrealistic, need to redo.
Parts:
- D3, D4: footprint Diode_SMD:D_0603_1608Metric -> Diode_SMD:D_SOD-123
Connections:
- net +3.3V: now also J4.2 (Pin_2)
- net +5V: no longer J4.2 (Pin_2)
Changed lines of the file:
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@@
     (property "Reference" "D3" (id 0) (at 41.91 26.67 0))
     (property "Value" "1N5819" (id 1) (at 41.91 31.75 0))
-    (property "Footprint" "Diode_SMD:D_0603_1608Metric" (id 2) (at 45.72 24.765 0)
+    (property "Footprint" "Diode_SMD:D_SOD-123" (id 2) (at 45.72 24.765 0)
       (effects (font (size 1.27 1.27)) hide)
     )
@@
     (property "Reference" "D4" (id 0) (at 64.77 26.67 0))
     (property "Value" "1N5819" (id 1) (at 64.77 31.75 0))
-    (property "Footprint" "Diode_SMD:D_0603_1608Metric" (id 2) (at 68.58 24.765 0)
+    (property "Footprint" "Diode_SMD:D_SOD-123" (id 2) (at 68.58 24.765 0)
       (effects (font (size 1.27 1.27)) hide)
     )
@@
     (pin "1")
     (pin "2")
-  )
-  (symbol (lib_id "power:+5V") (at 66.04 157.48 0) (unit 1)
-    (in_bom yes) (on_board yes) (fields_autoplaced)
-    (property "Reference" "#PWR060" (id 0) (at 66.04 161.29 0)
-      (effects (font (size 1.27 1.27)) hide)
-    )
-    (property "Value" "+5V" (id 1) (at 66.04 152.4 0))
-    (property "Footprint" "" (id 2) (at 66.04 157.48 0)
-      (effects (font (size 1.27 1.27)) hide)
-    )
-    (property "Datasheet" "" (id 3) (at 66.04 157.48 0)
-      (effects (font (size 1.27 1.27)) hide)
-    )
-    (pin "1")
   )
   (symbol (lib_id "power:+3.3V") (at 76.2 29.21 270) (unit 1)
@@
     (pin "1")
   )
+  (symbol (lib_id "power:+3.3V") (at 66.04 157.48 0) (unit 1)
+    (in_bom yes) (on_board yes)
+    (property "Reference" "#PWR0101" (id 0) (at 66.04 161.29 0)
+      (effects (font (size 1.27 1.27)) hide)
+    )
+    (property "Value" "+3.3V" (id 1) (at 64.77 153.67 0))
+    (property "Footprint" "" (id 2) (at 66.04 157.48 0)
+      (effects (font (size 1.27 1.27)) hide)
+    )
+    (property "Datasheet" "" (id 3) (at 66.04 157.48 0)
+      (effects (font (size 1.27 1.27)) hide)
+    )
+    (pin "1")
+  )
   (symbol (lib_id "Device:R") (at 71.12 161.29 270) (unit 1)
     (in_bom yes) (on_board yes)
@@
       (reference "#PWR059") (unit 1) (value "GND") (footprint "")
     )
-    (path "/7d8f4ff6-4c14-4fa6-8737-15c886f41213"
-      (reference "#PWR060") (unit 1) (value "+5V") (footprint "")
-    )
     (path "/cf7d19f3-5b44-44d1-aa39-e4fe47b8eb5b"
       (reference "#PWR061") (unit 1) (value "+3.3V") (footprint "")
@@
       (reference "#PWR078") (unit 1) (value "+3.3V") (footprint "")
     )
+    (path "/ee491e58-2553-4a50-822a-da4997d54c81"
+      (reference "#PWR0101") (unit 1) (value "+3.3V") (footprint "")
+    )
     (path "/95515899-f309-4706-b478-ef0c1d74de3d/6e926fcb-bc57-4a6a-ac9a-7920661fd921"
       (reference "C1") (unit 1) (value "4.7u") (footprint "Capacitor_SMD:C_0603_1608Metric")
@@
     )
     (path "/4dcd2554-0c0c-4fca-b220-d2fb156d9cf9/2194da5e-abcb-490c-ad12-09330a88057c"
-      (reference "D1") (unit 1) (value "1N5819") (footprint "Diode_SMD:D_0603_1608Metric")
+      (reference "D1") (unit 1) (value "1N5819") (footprint "Diode_SMD:D_SOD-123")
     )
     (path "/8c1d7bfe-a7ad-4b08-9e6d-dd7b239bc0ed/2194da5e-abcb-490c-ad12-09330a88057c"
-      (reference "D2") (unit 1) (value "1N5819") (footprint "Diode_SMD:D_0603_1608Metric")
+      (reference "D2") (unit 1) (value "1N5819") (footprint "Diode_SMD:D_SOD-123")
     )
     (path "/3c103bef-0efb-4142-b313-3083a43ce99d"
-      (reference "D3") (unit 1) (value "1N5819") (footprint "Diode_SMD:D_0603_1608Metric")
+      (reference "D3") (unit 1) (value "1N5819") (footprint "Diode_SMD:D_SOD-123")
     )
     (path "/7c2a1523-547e-41f9-846d-b97ecea82980"
-      (reference "D4") (unit 1) (value "1N5819") (footprint "Diode_SMD:D_0603_1608Metric")
+      (reference "D4") (unit 1) (value "1N5819") (footprint "Diode_SMD:D_SOD-123")
     )
     (path "/5098eb75-ab3f-49e8-b692-4372bb393d18"
