File: electrium-esc/MCU.kicad_sch (KiCad schematic)
At the start: 31 parts

Commit message: Prototype (almost) finished
Have to do electric check rules
Connections:
- net MISO_B: now also U?.75 (PB14); no longer U?.42 (PA6_(MISO))
- net MOSI_B: now also U?.76 (PB15); no longer U?.43 (PA7_(MOSI))
- net NRF_CE: now also U?.40 (PA4); no longer U?.74 (PB13)
- net NRF_CSN: now also U?.37 (PA3); no longer U?.73 (PB12)
- net NRF_MISO: now also U?.42 (PA6_(MISO)); no longer U?.75 (PB14)
- net NRF_MOSI: now also U?.43 (PA7_(MOSI)); no longer U?.76 (PB15)
- net NRF_SCK: now also U?.41 (PA5_(SCK)); no longer U?.69 (PB10)
- net SCK_B: now also U?.69 (PB10); no longer U?.41 (PA5_(SCK))
- net CS_A: now reaches U?.110 (PA15)
- net LED: now reaches U?.137 (PB7)
- new net CS_B: U?.74 (PB13)
- no-connect marks 60 -> 57
Changed lines of the file:
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@@
   (no_connect (at 73.66 186.69))
   (no_connect (at 73.66 156.21))
-  (no_connect (at 134.62 100.33))
   (no_connect (at 134.62 186.69))
-  (no_connect (at 134.62 72.39))
   (no_connect (at 73.66 194.31))
   (no_connect (at 134.62 196.85))
@@
   (no_connect (at 73.66 138.43))
   (no_connect (at 134.62 201.93))
+  (no_connect (at 134.62 135.89))
   (no_connect (at 134.62 125.73))
   (no_connect (at 73.66 184.15))
   (no_connect (at 73.66 176.53))
   (no_connect (at 134.62 219.71))
-  (no_connect (at 134.62 123.19))
   (no_connect (at 73.66 130.81))
   (no_connect (at 73.66 212.09))
@@
   (no_connect (at 134.62 82.55))
   (no_connect (at 134.62 87.63))
-  (no_connect (at 134.62 69.85))
   (no_connect (at 73.66 128.27))
   (wire (pts (xy 93.98 53.34) (xy 93.98 54.61))
@@
     )
   )
+  (hierarchical_label "CS_A" (shape output) (at 134.62 100.33 0)
+    (effects (font (size 1.27 1.27)) (justify left))
+  )
   (hierarchical_label "H1_B" (shape output) (at 73.66 227.33 180)
     (effects (font (size 1.27 1.27)) (justify right))
@@
     (effects (font (size 1.27 1.27)) (justify right))
   )
-  (hierarchical_label "NRF_CE" (shape output) (at 134.62 138.43 0)
+  (hierarchical_label "NRF_CE" (shape output) (at 134.62 72.39 0)
     (effects (font (size 1.27 1.27)) (justify left))
   )
@@
     (effects (font (size 1.27 1.27)) (justify right))
   )
+  (hierarchical_label "CS_B" (shape output) (at 134.62 138.43 0)
+    (effects (font (size 1.27 1.27)) (justify left))
+  )
   (hierarchical_label "L3_B" (shape output) (at 134.62 105.41 0)
     (effects (font (size 1.27 1.27)) (justify left))
@@
     (effects (font (size 1.27 1.27)) (justify right))
   )
-  (hierarchical_label "MISO_B" (shape input) (at 134.62 77.47 0)
+  (hierarchical_label "MISO_B" (shape input) (at 134.62 140.97 0)
     (effects (font (size 1.27 1.27)) (justify left))
   )
@@
     (effects (font (size 1.27 1.27)) (justify left))
   )
-  (hierarchical_label "NRF_MISO" (shape input) (at 134.62 140.97 0)
+  (hierarchical_label "NRF_MISO" (shape input) (at 134.62 77.47 0)
     (effects (font (size 1.27 1.27)) (justify left))
   )
@@
     (effects (font (size 1.27 1.27)) (justify right))
   )
-  (hierarchical_label "MOSI_B" (shape output) (at 134.62 80.01 0)
-    (effects (font (size 1.27 1.27)) (justify left))
-  )
-  (hierarchical_label "NRF_CSN" (shape output) (at 134.62 135.89 0)
+  (hierarchical_label "MOSI_B" (shape output) (at 134.62 143.51 0)
+    (effects (font (size 1.27 1.27)) (justify left))
+  )
+  (hierarchical_label "NRF_CSN" (shape output) (at 134.62 69.85 0)
     (effects (font (size 1.27 1.27)) (justify left))
   )
@@
     (effects (font (size 1.27 1.27)) (justify right))
   )
-  (hierarchical_label "SCK_B" (shape output) (at 134.62 74.93 0)
+  (hierarchical_label "SCK_B" (shape output) (at 134.62 130.81 0)
     (effects (font (size 1.27 1.27)) (justify left))
   )
@@
     (effects (font (size 1.27 1.27)) (justify left))
   )
-  (hierarchical_label "NRF_MOSI" (shape output) (at 134.62 143.51 0)
+  (hierarchical_label "NRF_MOSI" (shape output) (at 134.62 80.01 0)
     (effects (font (size 1.27 1.27)) (justify left))
   )
@@
     (effects (font (size 1.27 1.27)) (justify left))
   )
-  (hierarchical_label "NRF_SCK" (shape output) (at 134.62 130.81 0)
-    (effects (font (size 1.27 1.27)) (justify left))
-  )
+  (hierarchical_label "LED" (shape output) (at 134.62 123.19 0)
+    (effects (font (size 1.27 1.27)) (justify left))
+  )
+  (hierarchical_label "NRF_SCK" (shape output) (at 134.62 74.93 0)
+    (effects (font (size 1.27 1.27)) (justify left))
+  )

Commit message: Fix Error
Parts:
- C10, C11, C12, C13, C14, C15, C16, C17, C18, C19, C2, C20, C21, C22, C23, C24, C25, C3, C4, C5, C6, C7, C8, C9: renamed from C?; footprint (none) -> Capacitor_SMD:C_0603_1608Metric
- FB1: renamed from FB?; footprint (none) -> Ferrite_THT:LairdTech_28C0236-0JW-10
- J5: renamed from J?; footprint (none) -> Connector_PinHeader_2.54mm:PinHeader_1x06_P2.54mm_Horizontal
- R15: renamed from R?; footprint (none) -> Resistor_SMD:R_0603_1608Metric
- SW1: renamed from SW?; footprint (none) -> Resistor_SMD:R_0603_1608Metric
- Y1: renamed from Y?; footprint (none) -> Oscillator:Oscillator_SMD_TXC_7C-4Pin_5.0x3.2mm
- gave numbers to parts that had none: 2
Connections:
- no-connect marks 57 -> 58

Commit message: Update Footprints for schematic symbols
Parts:
- PS1: footprint SOT230P700X180-4N -> Package_TO_SOT_SMD:SOT-223
Changed lines of the file:
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@@
     (property "Reference" "PS1" (id 0) (at 44.45 20.32 0))
     (property "Value" "TC2117-3.3VDBTR" (id 1) (at 44.45 22.86 0))
-    (property "Footprint" "SOT230P700X180-4N" (id 2) (at 57.15 25.4 0)
+    (property "Footprint" "Package_TO_SOT_SMD:SOT-223" (id 2) (at 57.15 25.4 0)
       (effects (font (size 1.27 1.27)) (justify left) hide)
     )
