File: electrium-esc/Temp-Sens.kicad_sch (KiCad schematic)
At the start: 6 parts

Commit message: relabel components to make more sense
Parts:
- renumbered C75 to C76, C76 to C77, R60 to R71, R61 to R72
Changed lines of the file:
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@@
   (symbol (lib_id "power:GND") (at 153.67 118.11 0) (unit 1)
     (in_bom yes) (on_board yes) (fields_autoplaced)
-    (property "Reference" "#PWR0169" (id 0) (at 153.67 124.46 0)
+    (property "Reference" "#PWR076" (id 0) (at 153.67 124.46 0)
       (effects (font (size 1.27 1.27)) hide)
     )
@@
   (symbol (lib_id "Device:R") (at 153.67 109.22 0) (unit 1)
     (in_bom yes) (on_board yes) (fields_autoplaced)
-    (property "Reference" "R60" (id 0) (at 156.21 107.9499 0)
+    (property "Reference" "R71" (id 0) (at 156.21 107.9499 0)
       (effects (font (size 1.27 1.27)) (justify left))
     )
@@
   (symbol (lib_id "Device:C") (at 179.07 109.22 0) (unit 1)
     (in_bom yes) (on_board yes)
-    (property "Reference" "C76" (id 0) (at 181.61 107.95 0)
+    (property "Reference" "C77" (id 0) (at 181.61 107.95 0)
       (effects (font (size 1.27 1.27)) (justify left))
     )
@@
   (symbol (lib_id "power:GND") (at 187.96 118.11 0) (unit 1)
     (in_bom yes) (on_board yes) (fields_autoplaced)
-    (property "Reference" "#PWR0167" (id 0) (at 187.96 124.46 0)
+    (property "Reference" "#PWR077" (id 0) (at 187.96 124.46 0)
       (effects (font (size 1.27 1.27)) hide)
     )
@@
   (symbol (lib_id "power:+3.3V") (at 153.67 88.9 0) (unit 1)
     (in_bom yes) (on_board yes) (fields_autoplaced)
-    (property "Reference" "#PWR0168" (id 0) (at 153.67 92.71 0)
+    (property "Reference" "#PWR074" (id 0) (at 153.67 92.71 0)
       (effects (font (size 1.27 1.27)) hide)
     )
@@
   (symbol (lib_id "power:+3.3V") (at 187.96 88.9 0) (unit 1)
     (in_bom yes) (on_board yes) (fields_autoplaced)
-    (property "Reference" "#PWR0170" (id 0) (at 187.96 92.71 0)
+    (property "Reference" "#PWR075" (id 0) (at 187.96 92.71 0)
       (effects (font (size 1.27 1.27)) hide)
     )
@@
   (symbol (lib_id "Device:C") (at 144.78 109.22 0) (unit 1)
     (in_bom yes) (on_board yes)
-    (property "Reference" "C75" (id 0) (at 147.32 107.95 0)
+    (property "Reference" "C76" (id 0) (at 147.32 107.95 0)
       (effects (font (size 1.27 1.27)) (justify left))
     )
@@
   (symbol (lib_id "Device:R") (at 187.96 109.22 0) (unit 1)
     (in_bom yes) (on_board yes) (fields_autoplaced)
-    (property "Reference" "R61" (id 0) (at 190.5 107.9499 0)
+    (property "Reference" "R72" (id 0) (at 190.5 107.9499 0)
       (effects (font (size 1.27 1.27)) (justify left))
     )
